File: find-wire/find-wire.kicad_pcb (KiCad board)
At the start: 2 copper layers, 48 parts, among them Q1 BC548, Q2 BC558, SW1 SW_SPST, SW2 SW_SPST, U1 CD4060BE, U2 4001, U3 TLC271IP, U4 TDA2822M

Commit message: [find-wire] Finish
Routing:
- net (no net): vias 8 -> 0
Other:
- board outline added: 84.8 x 136 mm
Changed lines of the file:
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@@
   (general
     (thickness 1.6)
-    (drawings 12)
-    (tracks 196)
+    (drawings 20)
+    (tracks 188)
     (zones 0)
     (modules 48)
@@
   )
   (setup
-    (last_trace_width 1)
+    (last_trace_width 0.25)
     (user_trace_width 1)
     (user_trace_width 1.27)
@@
     (uvia_drill 0.1)
     (uvias_allowed no)
-    (uvia_min_size 0.2)
+    (uvia_min_size 0.3)
     (uvia_min_drill 0.1)
     (edge_width 0.1)
@@
     (visible_elements FFFFFF7F)
     (pcbplotparams
-      (layerselection 0x00000_fffffffe)
+      (layerselection 0x010f0_ffffffff)
       (usegerberextensions false)
       (usegerberattributes false)
@@
       (padsonsilk false)
       (subtractmaskfromsilk false)
-      (outputformat 2)
+      (outputformat 1)
       (mirror false)
-      (drillshape 1)
+      (drillshape 0)
       (scaleselection 1)
       (outputdirectory "output"))
@@
     (tags connector)
     (attr virtual)
-    (fp_text reference RV1 (at 7.62 -5.08 90) (layer F.SilkS)
+    (fp_text reference RV1 (at -6.5 -0.25 90) (layer F.SilkS)
       (effects (font (size 1 1) (thickness 0.15)))
     )
@@
     (descr "LED, diameter 3.0mm, 2 pins")
     (tags "LED diameter 3.0mm 2 pins")
-    (fp_text reference D1 (at 1.27 -2.96) (layer F.SilkS)
+    (fp_text reference D1 (at -3.5 0) (layer F.SilkS)
       (effects (font (size 1 1) (thickness 0.15)))
     )
@@
     (descr "C, Disc series, Radial, pin pitch=5.00mm, , diameter*width=4.3*1.9mm^2, Capacitor, http://www.vishay.com/docs/45233/krseries.pdf")
     (tags "C Disc series Radial pin pitch 5.00mm  diameter 4.3mm width 1.9mm Capacitor")
-    (fp_text reference C4 (at 2.5 -2.2 90) (layer F.SilkS)
+    (fp_text reference C4 (at 2.25 3 90) (layer F.SilkS)
       (effects (font (size 1 1) (thickness 0.15)))
     )
@@
     (descr "C, Disc series, Radial, pin pitch=5.00mm, , diameter*width=10*2.5mm^2, Capacitor, http://cdn-reichelt.de/documents/datenblatt/B300/DS_KERKO_TC.pdf")
     (tags "C Disc series Radial pin pitch 5.00mm  diameter 10mm width 2.5mm Capacitor")
-    (fp_text reference C1 (at 2.5 -2.5) (layer F.SilkS)
+    (fp_text reference C1 (at -4.5 -0.25) (layer F.SilkS)
       (effects (font (size 1 1) (thickness 0.15)))
     )
@@
     (tags connector)
     (attr virtual)
-    (fp_text reference BT2 (at 3.81 -5.08) (layer F.SilkS)
+    (fp_text reference BT2 (at -7 -0.75) (layer F.SilkS)
       (effects (font (size 1 1) (thickness 0.15)))
     )
@@
       (net 1 "Net-(AE1-Pad1)"))
   )
+  (gr_line (start 121 111.5) (end 121 154) (layer Edge.Cuts) (width 0.1))
+  (gr_line (start 36.25 111.5) (end 121 111.5) (layer Edge.Cuts) (width 0.1))
+  (gr_line (start 36.25 154) (end 36.25 111.5) (layer Edge.Cuts) (width 0.1))
+  (gr_line (start 121 154) (end 36.25 154) (layer Edge.Cuts) (width 0.1))
+  (gr_line (start 111.75 18) (end 111.75 88.5) (layer Edge.Cuts) (width 0.1))
+  (gr_line (start 39.25 18) (end 111.75 18) (layer Edge.Cuts) (width 0.1))
+  (gr_line (start 39.25 88.5) (end 39.25 18) (layer Edge.Cuts) (width 0.1))
+  (gr_line (start 111.75 88.5) (end 39.25 88.5) (layer Edge.Cuts) (width 0.1))
   (gr_text "DETECTOR\nFRONT" (at 105 21.75) (layer F.Cu)
     (effects (font (size 1.5 1.5) (thickness 0.3)))
@@
     (effects (font (size 1.5 1.5) (thickness 0.3)) (justify mirror))
   )
-  (via (at 34.5 110.25) (size 2) (drill 1) (layers F.Cu B.Cu) (net 0))
-  (via (at 34.5 155) (size 2) (drill 1) (layers F.Cu B.Cu) (net 0))
-  (via (at 122.5 155) (size 2) (drill 1) (layers F.Cu B.Cu) (net 0))
-  (via (at 122.5 110.25) (size 2) (drill 1) (layers F.Cu B.Cu) (net 0))
-  (via (at 38 90) (size 2) (drill 1) (layers F.Cu B.Cu) (net 0))
-  (via (at 38 17) (size 2) (drill 1) (layers F.Cu B.Cu) (net 0))
-  (via (at 114.25 90) (size 2) (drill 1) (layers F.Cu B.Cu) (net 0))
-  (via (at 114.25 17) (size 2) (drill 1) (layers F.Cu B.Cu) (net 0))
   (segment (start 61.445212 38) (end 61.468893 37.976319) (width 2) (layer F.Cu) (net 1))
   (segment (start 44.5 38) (end 61.445212 38) (width 2) (layer F.Cu) (net 1))
