File: light/light.sch (KiCad schematic (older format))
At the start: 55 parts, among them J1 Conn_01x02_Female, J10 Conn_01x02_Female, J11 Conn_01x02_Male, J12 Conn_01x02_Female, J13 Conn_01x02_Female, J14 Conn_01x02_Male, J15 Conn_01x02_Female, J16 Conn_01x02_Female, J17 Conn_01x02_Male, J18 Conn_01x02_Female, J19 Conn_01x02_Female, J2 Conn_02x08_Odd_Even, J20 Conn_01x02_Male, J21 Conn_01x02_Female, J22 Conn_01x02_Female, J23 Conn_01x02_Male, J24 Conn_01x02_Female, J25 Conn_01x02_Female, J26 Conn_01x02_Male, J3 Conn_01x02_Female, J4 Conn_01x02_Female, J5 Conn_01x02_Male, J6 Conn_01x02_Female, J7 Conn_01x02_Female, J8 Conn_01x02_Male, J9 Conn_01x02_Female, SW1 SW_SPST, U1 L7805, U10 LDB600, U2 TLC555CPS, U3 LDB600, U4 LDB600, U5 LDB600, U6 LDB600, U7 LDB600, U8 LDB600, U9 LDB600

Commit message: [light] Finish
Parts:
- added C_buf: 0.1u, symbol Device:C
- added U2_buf: 74HC125N, DIP254P762X420-14, symbol 74HC125N:74HC125N
- U2: symbol Timer:TLC555CPS -> light-rescue:TLC555CPS-Timer
Connections:
- net +5V: now also C_buf.1, U2_buf.14 (VCC)
- net GND: now also C_buf.2, U2_buf.1 (1~OE), U2_buf.10 (3~OE), U2_buf.13 (4~OE), U2_buf.4 (2~OE), U2_buf.7 (GND)
- net pwm_out: now also U2_buf.12 (4A), U2_buf.2 (1A), U2_buf.5 (2A), U2_buf.9 (3A); no longer J2.1 (Pin_1), J2.11 (Pin_11), J2.13 (Pin_13), J2.15 (Pin_15), J2.3 (Pin_3), J2.5 (Pin_5), J2.7 (Pin_7), J2.9 (Pin_9)
- new net: J2.1 (Pin_1), J2.3 (Pin_3), U2_buf.3 (1Y)
- new net: J2.11 (Pin_11), J2.9 (Pin_9), U2_buf.8 (3Y)
- new net: J2.13 (Pin_13), J2.15 (Pin_15), U2_buf.11 (4Y)
- new net: J2.5 (Pin_5), J2.7 (Pin_7), U2_buf.6 (2Y)
Other:
- moved on the sheet: J1, J2
