File: light/light.kicad_pcb (KiCad board)
At the start: 2 copper layers, 55 parts, among them J1 Conn_01x02_Female, J10 Conn_01x02_Female, J11 Conn_01x02_Male, J12 Conn_01x02_Female, J13 Conn_01x02_Female, J14 Conn_01x02_Male, J15 Conn_01x02_Female, J16 Conn_01x02_Female, J17 Conn_01x02_Male, J18 Conn_01x02_Female, J19 Conn_01x02_Female, J2 Conn_02x08_Odd_Even, J20 Conn_01x02_Male, J21 Conn_01x02_Female, J22 Conn_01x02_Female, J23 Conn_01x02_Male, J24 Conn_01x02_Female, J25 Conn_01x02_Female, J26 Conn_01x02_Male, J3 Conn_01x02_Female, J4 Conn_01x02_Female, J5 Conn_01x02_Male, J6 Conn_01x02_Female, J7 Conn_01x02_Female, J8 Conn_01x02_Male, J9 Conn_01x02_Female, SW1 SW_SPST, U1 L7805, U10 LDB600, U2 TLC555CPS, U3 LDB600, U4 LDB600, U5 LDB600, U6 LDB600, U7 LDB600, U8 LDB600, U9 LDB600

Commit message: [ligh] Finish
Parts:
- moved U7 375.8 mm to (266.0, 39.8)
- moved J13 346.4 mm to (199.2, 44.5), turned to 270 degrees
- moved U10 320.1 mm to (266.0, 108.5)
- moved J17 307.3 mm to (262.2, 61.5)
- moved J26 305.2 mm to (262.2, 130.2)
- moved U6 303.6 mm to (216.0, 39.8)
- moved U9 293.7 mm to (216.0, 108.5)
- moved U5 292.4 mm to (159.8, 39.8)
- moved J24 278.4 mm to (244.0, 103.8), turned to 90 degrees
- moved J25 272.7 mm to (249.2, 113.2), turned to 270 degrees
- moved J12 270.2 mm to (194.0, 35.0), turned to 90 degrees
- moved C13 269.2 mm to (251.8, 96.2), turned to 270 degrees
- moved J14 268.7 mm to (212.2, 61.5)
- moved C10 267.1 mm to (251.8, 27.5), turned to 270 degrees
- moved J23 263.1 mm to (212.2, 130.2)
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Connections:
- J9 pad 2: Net-(C8-Pad1) -> (no net)
Routing:
- net Net-(J4-Pad2): track 0.00 -> 35.8 mm
- net Net-(J22-Pad2): track 0.00 -> 35.8 mm
- net Net-(J19-Pad2): track 0.00 -> 35.8 mm
- net Net-(J7-Pad2): track 0.00 -> 35.8 mm
- net Net-(J25-Pad2): track 0.00 -> 35.8 mm
- net Net-(J13-Pad2): track 0.00 -> 35.8 mm
- net Net-(J10-Pad2): track 0.00 -> 35.8 mm
- net Net-(J16-Pad2): track 0.00 -> 35.8 mm
- net Net-(C9-Pad2): track 0.00 -> 20.5 mm
- net Net-(C8-Pad2): track 0.00 -> 20.5 mm
- net Net-(C7-Pad2): track 0.00 -> 20.5 mm
- net Net-(C6-Pad2): track 0.00 -> 20.5 mm
- net Net-(C13-Pad2): track 0.00 -> 20.5 mm
- net Net-(C12-Pad2): track 0.00 -> 20.5 mm
- net Net-(C11-Pad2): track 0.00 -> 20.5 mm
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- added copper zone on F.Cu, net (none)
- added copper zone on B.Cu, net Net-(C10-Pad1)
- added copper zone on B.Cu, net Net-(C10-Pad2)
- added copper zone on B.Cu, net Net-(C11-Pad1)
- added copper zone on B.Cu, net Net-(C11-Pad2)
- added copper zone on B.Cu, net Net-(C12-Pad1)
- added copper zone on B.Cu, net Net-(C12-Pad2)
- added copper zone on B.Cu, net Net-(C13-Pad1)
- added copper zone on B.Cu, net Net-(C13-Pad2)
- added copper zone on B.Cu, net Net-(C6-Pad1)
- added copper zone on B.Cu, net Net-(C6-Pad2)
- added copper zone on B.Cu, net Net-(C7-Pad1)
- added copper zone on B.Cu, net Net-(C7-Pad2)
- added copper zone on B.Cu, net Net-(C8-Pad1)
- added copper zone on B.Cu, net Net-(C8-Pad2)
- added copper zone on B.Cu, net Net-(C9-Pad1)
- added copper zone on B.Cu, net Net-(C9-Pad2)
- added copper zone on B.Cu, net Net-(J11-Pad1)
- added copper zone on B.Cu, net Net-(J11-Pad2)
- added copper zone on B.Cu, net Net-(J14-Pad1)
- added copper zone on B.Cu, net Net-(J14-Pad2)
- added copper zone on B.Cu, net Net-(J17-Pad1)
- added copper zone on B.Cu, net Net-(J17-Pad2)
- added copper zone on B.Cu, net Net-(J20-Pad1)
- added copper zone on B.Cu, net Net-(J20-Pad2)
- added copper zone on B.Cu, net Net-(J23-Pad1)
- added copper zone on B.Cu, net Net-(J23-Pad2)
- added copper zone on B.Cu, net Net-(J26-Pad1)
- added copper zone on B.Cu, net Net-(J26-Pad2)
- added copper zone on B.Cu, net Net-(J5-Pad1)
- added copper zone on B.Cu, net Net-(J5-Pad2)
- added copper zone on B.Cu, net Net-(J8-Pad1)
- added copper zone on B.Cu, net Net-(J8-Pad2)
Other:
- board text added: "+12V SW"
- board text added: "BACK"
- board text added: "FRONT"
- board text added: "GND +12V"
- board text added: "OUT - +"
- board text added: "PWM GND"
- board text removed: "GND SIG"
- board text removed: "SW +12V"

Commit message: [light] Finish
Routing:
- net (no net): vias 36 -> 0
Other:
- board outline added: 252.5 x 168.8 mm

Commit message: [light] update
Parts:
- added U2_buf1: 74HC125N, LIB:DIP254P762X420-14, F.Cu at (135.5, 131.7)
Connections:
- J2 pad 1: /pwm_out -> Net-(J2-Pad1)
- J2 pad 11: /pwm_out -> Net-(J2-Pad11)
- J2 pad 13: /pwm_out -> Net-(J2-Pad13)
- J2 pad 15: /pwm_out -> Net-(J2-Pad13)
- J2 pad 3: /pwm_out -> Net-(J2-Pad1)
- J2 pad 5: /pwm_out -> Net-(J2-Pad5)
- J2 pad 7: /pwm_out -> Net-(J2-Pad5)
- J2 pad 9: /pwm_out -> Net-(J2-Pad11)
- J9 pad 2: (no net) -> Net-(C8-Pad1)
- R3 pad 1: Net-(R3-Pad1) -> Net-(RV1-Pad1)
- RV1 pad 1: Net-(R2-Pad2) -> Net-(RV1-Pad1)
- RV1 pad 3: Net-(R3-Pad1) -> Net-(R2-Pad2)
- U2 pad 5: (no net) -> unconnected-(U2-Pad5)
Routing:
- net Net-(J2-Pad11): track 0.00 -> 23.7 mm
- net /pwm_out: track 23.7 -> 0.00 mm
- net Net-(RV1-Pad1): track 0.00 -> 9.63 mm
- net Net-(R3-Pad1): track 9.63 -> 0.00 mm
Other:
- net class Default removed
