File: spot-welding/spot-welding.kicad_sch (KiCad schematic)
At the start: 32 parts, among them J1 Conn_01x01_Female, J2 Conn_01x01_Female, K1 R, K1.1 SW_SPST, K2 R_Potentiometer, K2.1 SW_SPST, M1 Fan, P1 Conn_WallPlug, SW1 SW_SPST, SW2 SW_SPDT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

Commit message: [spot-welding] update
Parts:
- H1, H2, H3: value (none) -> Lamp
- K1: value (none) -> R
- M1: value (none) -> Fan
- P1: value (none) -> Conn_WallPlug
- SW2: value (none) -> SW_DPDT_x2
- SW3: value (none) -> SW_Push
- gave numbers to parts that had none: 2
Changed lines of the file:
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@@
       (effects (font (size 1.27 1.27)) (justify left))
     )
-    (property "Value" "" (id 1) (at 175.895 121.0822 0)
+    (property "Value" "Lamp" (id 1) (at 175.895 121.0822 0)
       (effects (font (size 1.27 1.27)) (justify left) hide)
     )
@@
   (symbol (lib_name "Conn_01x01_Female_1") (lib_id "Connector:Conn_01x01_Female") (at 270.51 146.05 0) (unit 1)
     (in_bom yes) (on_board yes) (fields_autoplaced)
-    (property "Reference" "J?" (id 0) (at 271.2212 145.2153 0)
+    (property "Reference" "J1" (id 0) (at 271.78 146.0499 0)
       (effects (font (size 1.27 1.27)) (justify left))
     )
@@
     (in_bom yes) (on_board yes) (fields_autoplaced)
     (property "Reference" "SW3" (id 0) (at 128.27 92.4392 0))
-    (property "Value" "" (id 1) (at 128.27 94.9761 0)
+    (property "Value" "SW_Push" (id 1) (at 128.27 94.9761 0)
       (effects (font (size 1.27 1.27)) hide)
     )
@@
       (effects (font (size 1.27 1.27)) (justify left))
     )
-    (property "Value" "" (id 1) (at 233.045 152.8322 0)
+    (property "Value" "Lamp" (id 1) (at 233.045 152.8322 0)
       (effects (font (size 1.27 1.27)) (justify left) hide)
     )
@@
       (effects (font (size 1.27 1.27)) (justify left))
     )
-    (property "Value" "" (id 1) (at 96.7232 121.0822 0)
+    (property "Value" "Fan" (id 1) (at 96.7232 121.0822 0)
       (effects (font (size 1.27 1.27)) (justify left) hide)
     )
@@
     (in_bom yes) (on_board yes)
     (property "Reference" "SW2" (id 0) (at 125.73 137.4308 0))
-    (property "Value" "" (id 1) (at 125.73 134.8939 0)
+    (property "Value" "SW_DPDT_x2" (id 1) (at 125.73 134.8939 0)
       (effects (font (size 1.27 1.27)) hide)
     )
@@
       (effects (font (size 1.27 1.27)) (justify left))
     )
-    (property "Value" "" (id 1) (at 187.198 119.8122 0)
+    (property "Value" "R" (id 1) (at 187.198 119.8122 0)
       (effects (font (size 1.27 1.27)) (justify left) hide)
     )
@@
     (in_bom yes) (on_board yes) (fields_autoplaced)
     (property "Reference" "SW2" (id 0) (at 125.73 102.5992 0))
-    (property "Value" "" (id 1) (at 125.73 105.1361 0)
+    (property "Value" "SW_DPDT_x2" (id 1) (at 125.73 105.1361 0)
       (effects (font (size 1.27 1.27)) hide)
     )
@@
   (symbol (lib_id "Connector:Conn_01x01_Female") (at 270.51 156.21 0) (unit 1)
     (in_bom yes) (on_board yes) (fields_autoplaced)
-    (property "Reference" "J?" (id 0) (at 271.2212 155.3753 0)
+    (property "Reference" "J2" (id 0) (at 271.78 156.2099 0)
       (effects (font (size 1.27 1.27)) (justify left))
     )
@@
       (effects (font (size 1.27 1.27)) (justify left))
     )
-    (property "Value" "" (id 1) (at 81.915 118.5422 0)
+    (property "Value" "Lamp" (id 1) (at 81.915 118.5422 0)
       (effects (font (size 1.27 1.27)) (justify left) hide)
     )
@@
     (in_bom yes) (on_board yes) (fields_autoplaced)
     (property "Reference" "P1" (id 0) (at 33.2105 104.2502 0))
-    (property "Value" "" (id 1) (at 33.2105 106.7871 0)
+    (property "Value" "Conn_WallPlug" (id 1) (at 33.2105 106.7871 0)
       (effects (font (size 1.27 1.27)) hide)
     )
@@
       (reference "H3") (unit 1) (value "Lamp") (footprint "")
     )
+    (path "/49455629-6bb1-4ec3-9275-a337b94b62f4"
+      (reference "J1") (unit 1) (value "Conn_01x01_Female") (footprint "")
+    )
     (path "/cbd460f0-34e5-4e3a-83f9-902bd31de4b9"
       (reference "J1") (unit 1) (value "Conn_01x01_Female") (footprint "")
@@
       (reference "J2") (unit 1) (value "Conn_01x01_Female") (footprint "")
     )
-    (path "/49455629-6bb1-4ec3-9275-a337b94b62f4"
-      (reference "J?") (unit 1) (value "Conn_01x01_Female") (footprint "")
-    )
     (path "/e525bce2-fe1f-4ac3-80f6-aeb7cb7b3601"
-      (reference "J?") (unit 1) (value "Conn_01x01_Female") (footprint "")
+      (reference "J2") (unit 1) (value "Conn_01x01_Female") (footprint "")
     )
     (path "/666dca55-a12c-405c-9cb8-6e3263091851"
