File: soft-start/soft-start.kicad_pcb (KiCad board)
At the start: 2 copper layers, 56.5 x 48.9 mm, 28 parts, among them Q1 IRFB3004PbF, U1 4011, U2 CD4060BE

Commit message: [DRL] [soft-start] Update track widths. Prepare for plotting
Changed lines of the file:
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@@
     (pad_to_mask_clearance 0)
     (pcbplotparams
-      (layerselection 0x00010fc_ffffffff)
+      (layerselection 0x0000000_fffffffe)
       (plot_on_all_layers_selection 0x0000000_00000000)
       (disableapertmacros false)
@@
       (sketchpadsonfab false)
       (subtractmaskfromsilk false)
-      (outputformat 1)
-      (mirror false)
+      (outputformat 2)
+      (mirror true)
       (drillshape 1)
       (scaleselection 1)
-      (outputdirectory "")
+      (outputdirectory "output")
     )
   )
@@
     (fp_circle (center 7.8 0) (end 9.75 0)
       (stroke (width 0.1) (type solid)) (fill none) (layer "F.Fab"))
-    (pad "1" thru_hole roundrect (at 0 0) (size 3.9 3.9) (drill 2.1) (layers "*.Cu" "*.Mask") (roundrect_rratio 0.064103)
+    (pad "1" thru_hole roundrect (at 0 0) (size 3.9 3.9) (drill 2.1) (layers "*.Cu" "*.Mask") (roundrect_rratio 0.06410307692)
       (net 9 "Net-(D2-A2)") (pinfunction "A") (pintype "passive"))
     (pad "2" thru_hole circle (at 7.8 0) (size 3.9 3.9) (drill 2.1) (layers "*.Cu" "*.Mask")
@@
     (fp_circle (center 6 0) (end 7.5 0)
       (stroke (width 0.1) (type solid)) (fill none) (layer "F.Fab"))
-    (pad "1" thru_hole roundrect (at 0 0) (size 3.1 3.1) (drill 2.1) (layers "*.Cu" "*.Mask") (roundrect_rratio 0.080645)
+    (pad "1" thru_hole roundrect (at 0 0) (size 3.1 3.1) (drill 2.1) (layers "*.Cu" "*.Mask") (roundrect_rratio 0.08064483871)
       (net 8 "+BATT") (pinfunction "-") (pintype "passive"))
     (pad "2" thru_hole circle (at 6 0) (size 3.1 3.1) (drill 2.1) (layers "*.Cu" "*.Mask")
@@
     (fp_line (start 5.625 5) (end 5.625 -5)
       (stroke (width 0.1) (type solid)) (layer "B.Fab"))
-    (pad "1" smd roundrect (at -7.65 2.54 90) (size 4.6 1.1) (layers "B.Cu" "B.Paste" "B.Mask") (roundrect_rratio 0.227273)
+    (pad "1" smd roundrect (at -7.65 2.54 90) (size 4.6 1.1) (layers "B.Cu" "B.Paste" "B.Mask") (roundrect_rratio 0.2272727273)
       (net 14 "/TRIGGER_OUT") (pinfunction "G") (pintype "input"))
-    (pad "2" smd roundrect (at -0.925 -2.775 90) (size 4.55 5.25) (layers "B.Cu" "B.Paste") (roundrect_rratio 0.054945)
+    (pad "2" smd roundrect (at -0.925 -2.775 90) (size 4.55 5.25) (layers "B.Cu" "B.Paste") (roundrect_rratio 0.05494505495)
       (net 9 "Net-(D2-A2)") (pinfunction "D") (pintype "passive"))
-    (pad "2" smd roundrect (at -0.925 2.775 90) (size 4.55 5.25) (layers "B.Cu" "B.Paste") (roundrect_rratio 0.054945)
+    (pad "2" smd roundrect (at -0.925 2.775 90) (size 4.55 5.25) (layers "B.Cu" "B.Paste") (roundrect_rratio 0.05494505495)
       (net 9 "Net-(D2-A2)") (pinfunction "D") (pintype "passive"))
-    (pad "2" smd roundrect (at 1.5 0 90) (size 9.4 10.8) (layers "B.Cu" "B.Mask") (roundrect_rratio 0.026596)
+    (pad "2" smd roundrect (at 1.5 0 90) (size 9.4 10.8) (layers "B.Cu" "B.Mask") (roundrect_rratio 0.02659595745)
       (net 9 "Net-(D2-A2)") (pinfunction "D") (pintype "passive"))
-    (pad "2" smd roundrect (at 3.925 -2.775 90) (size 4.55 5.25) (layers "B.Cu" "B.Paste") (roundrect_rratio 0.054945)
+    (pad "2" smd roundrect (at 3.925 -2.775 90) (size 4.55 5.25) (layers "B.Cu" "B.Paste") (roundrect_rratio 0.05494505495)
       (net 9 "Net-(D2-A2)") (pinfunction "D") (pintype "passive"))
-    (pad "2" smd roundrect (at 3.925 2.775 90) (size 4.55 5.25) (layers "B.Cu" "B.Paste") (roundrect_rratio 0.054945)
+    (pad "2" smd roundrect (at 3.925 2.775 90) (size 4.55 5.25) (layers "B.Cu" "B.Paste") (roundrect_rratio 0.05494505495)
       (net 9 "Net-(D2-A2)") (pinfunction "D") (pintype "passive"))
-    (pad "3" smd roundrect (at -7.65 -2.54 90) (size 4.6 1.1) (layers "B.Cu" "B.Paste" "B.Mask") (roundrect_rratio 0.227273)
+    (pad "3" smd roundrect (at -7.65 -2.54 90) (size 4.6 1.1) (layers "B.Cu" "B.Paste" "B.Mask") (roundrect_rratio 0.2272727273)
       (net 1 "GND") (pinfunction "S") (pintype "passive"))
     (model "${KICAD6_3DMODEL_DIR}/Package_TO_SOT_SMD.3dshapes/TO-263-2.wrl"
