File: adapter/adapter.kicad_sch (KiCad schematic)
At the start: 10 parts, among them Q1 IRFB3004PbF, Q2 AUIRF2804S, U1 IRS10752LPbF, U2 P0102BL, U3 TLC555xD, U4 TLC555xP, U5 TLC555xP, U6 EL814, U7 TLC555xP

Commit message: [adapter] Update PCB
Parts:
- U4: footprint Package_DIP:DIP-8_W7.62mm -> Package_DIP:DIP-8_W10.16mm
Changed lines of the file:
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@@
       (effects (font (size 1.27 1.27)) (justify left))
     )
-    (property "Footprint" "Package_DIP:DIP-8_W7.62mm" (at 216.535 153.035 0)
+    (property "Footprint" "Package_DIP:DIP-8_W10.16mm" (at 216.535 153.035 0)
       (effects (font (size 1.27 1.27)) hide)
     )
